Commit message: add positions

File: urdf/dynamixel.urdf (robot description, URDF)
Before this commit: robot arm, 5 links, 4 joints
Joints:
- removed joint base_to_torso
- removed joint torso_to_bone
- added joint base: type revolute, parent base, child torso, origin xyz=0 0 0.05, axis 0 0 1, limit lower=-1.57 upper=1.57 effort=1000.0 velocity=0.5
- added joint base_to_bone: type revolute, parent torso, child bone, origin xyz=-0.08 0 0.035, axis 0 1 0, limit lower=-1.57 upper=0.523 effort=1000.0 velocity=0.5
