Commit message: update

File: urdf/dynamixel (copy).urdf (robot description, URDF)
Before this commit: robot arm, 6 links, 5 joints
Links:
- removed link base_frame
- link bone: geometry visual box size=0.03 0.001 0.045; visual box size=0.03 0.001 0.045
Joints:
- removed joint world_base
- joint base: limit lower=1 upper=2 effort=1000.0 velocity=0.5 -> lower=-1.57 upper=1.57 effort=1000.0 velocity=0.5
- joint base_to_bone: limit lower=0 upper=2 effort=1000.0 velocity=0.5 -> lower=-1.57 upper=0.523 effort=1000.0 velocity=0.5
- joint bone_to_hand: limit lower=-2 upper=2 effort=1000.0 velocity=0.5 -> lower=-1.57 upper=1.57 effort=1000.0 velocity=0.5; origin xyz=-0.16 0 0 -> xyz=0 0 0.16
